File: DosingPCB/SD-Card.kicad_sch (KiCad schematic)
At the start: 11 parts, among them J1 Micro_SD_Card, U10 4050, U12 LP2985-3.3, U2 4050, U3 4050, U4 4050, U8 4050, U9 4050

Commit message: Basically finished schematic
Parts:
- removed U10, U2, U3, U4, U8: 4050, symbol 4xxx:4050
- removed U12: LP2985-3.3, Package_TO_SOT_SMD:SOT-23-5, symbol Regulator_Linear:LP2985-3.3
- removed U9: 4050, symbol 4xxx_IEEE:4050
- added U5: 4050, CD74HC4050MT:SOIC127P600X175-16N, symbol 4xxx_IEEE:4050
- C7: renamed from C1; footprint (none) -> Capacitor_SMD:C_0603_1608Metric
- D4: renamed from D1; value LED -> Red; footprint (none) -> LED_SMD:LED_0603_1608Metric
- J6: renamed from J1; footprint (none) -> Connector_Card:microSD_HC_Molex_104031-0811
- R8: renamed from R1; footprint (none) -> Resistor_SMD:R_0805_2012Metric
Connections:
- net +3.3V: now also U5.1 (Vdd), U5.1 (Vdd), U5.1 (Vdd), U5.1 (Vdd), U5.1 (Vdd), U5.1 (Vdd)
- net CLK: now also U5.3, U5.7
- net CS: now also U5.9
- net DataIn: now also U5.5
- net GND: now also U5.11, U5.14, U5.8 (Vss), U5.8 (Vss), U5.8 (Vss), U5.8 (Vss), U5.8 (Vss), U5.8 (Vss)
- net at J6.3 (CMD), R8.2: now also U5.10
- net at D4.2 (A): now also U5.2
- net at J6.8 (DAT1): now also U5.4
- net at J6.5 (CLK): now also U5.6
- net CD: now reaches J6.2 (DAT3/CD)
- no-connect marks 5 -> 3
Other:
- moved on the sheet: C7

Commit message: 98% completed PCB
Other:
- moved on the sheet: C7
Changed lines of the file:
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@@
+	)
+	(junction
+		(at 173.99 91.44)
+		(diameter 0)
+		(color 0 0 0 0)
 	)
 	(junction
@@
 	)
 	(symbol
+		(lib_id "power:PWR_FLAG")
+		(at 173.99 91.44 0)
+		(unit 1)
+		(body_style 1)
+		(exclude_from_sim no)
+		(in_bom yes)
+		(on_board yes)
+		(in_pos_files yes)
+		(dnp no)
+		(fields_autoplaced yes)
+		(property "Reference" "#FLG05"
+			(at 173.99 89.535 0)
+			(hide yes)
+			(show_name no)
+			(do_not_autoplace no)
+			(effects
+				(font
+					(size 1.27 1.27)
+				)
+			)
+		)
+		(property "Value" "PWR_FLAG"
+			(at 173.99 86.36 0)
+			(show_name no)
+			(do_not_autoplace no)
+			(effects
+				(font
+					(size 1.27 1.27)
+				)
+			)
+		)
+		(property "Footprint" ""
+			(at 173.99 91.44 0)
+			(hide yes)
+			(show_name no)
+			(do_not_autoplace no)
+			(effects
+				(font
+					(size 1.27 1.27)
+				)
+			)
+		)
+		(property "Datasheet" ""
+			(at 173.99 91.44 0)
+			(hide yes)
+			(show_name no)
+			(do_not_autoplace no)
+			(effects
+				(font
+					(size 1.27 1.27)
+				)
+			)
+		)
+		(property "Description" "Special symbol for telling ERC where power comes from"
+			(at 173.99 91.44 0)
+			(hide yes)
+			(show_name no)
+			(do_not_autoplace no)
+			(effects
+				(font
+					(size 1.27 1.27)
+				)
+			)
+		)
+		(pin "1"
+		)
+		(instances
+			(project "DosingPCB"
+				(path "/3d87c741-aedb-4217-929e-9b442255b4c1/b7875638-5f41-4a4c-aed1-479849be983a"
+					(reference "#FLG05")
+					(unit 1)
+				)
+			)
+		)
+	)
+	(symbol
 		(lib_id "Device:C")
-		(at 160.02 114.3 0)
+		(at 160.02 119.38 0)
 		(unit 1)
 		(body_style 1)
@@
 		(dnp no)
 		(property "Reference" "C7"
-			(at 163.576 114.3 90)
+			(at 163.576 119.38 90)
 			(show_name no)
 			(do_not_autoplace no)
@@
 		)
 		(property "Value" ".1uF"
-			(at 154.178 114.554 0)
+			(at 154.178 119.634 0)
 			(show_name no)
 			(do_not_autoplace no)
@@
 		)
 		(property "Footprint" "Capacitor_SMD:C_0603_1608Metric"
-			(at 160.9852 118.11 0)
+			(at 160.9852 123.19 0)
 			(hide yes)
 			(show_name no)
@@
 		)
 		(property "Datasheet" ""
-			(at 160.02 114.3 0)
+			(at 160.02 119.38 0)
 			(hide yes)
 			(show_name no)
@@
 		)
 		(property "Description" "Unpolarized capacitor"
-			(at 160.02 114.3 0)
+			(at 160.02 119.38 0)
 			(hide yes)
 			(show_name no)
@@
 	(symbol
 		(lib_id "power:GND")
-		(at 160.02 118.11 0)
+		(at 160.02 123.19 0)
 		(unit 1)
 		(body_style 1)
@@
 		(dnp no)
 		(property "Reference" "#PWR034"
-			(at 160.02 124.46 0)
+			(at 160.02 129.54 0)
 			(hide yes)
 			(show_name no)
@@
 		)
 		(property "Value" "GND"
-			(at 160.02 122.936 90)
+			(at 160.02 128.016 90)
 			(show_name no)
 			(do_not_autoplace no)
@@
 		)
 		(property "Footprint" ""
-			(at 160.02 118.11 0)
+			(at 160.02 123.19 0)
 			(hide yes)
 			(show_name no)
@@
 		)
 		(property "Datasheet" ""
-			(at 160.02 118.11 0)
+			(at 160.02 123.19 0)
 			(hide yes)
 			(show_name no)
@@
 		)
 		(property "Description" "Power symbol creates a global label with name \"GND\" , ground"
-			(at 160.02 118.11 0)
+			(at 160.02 123.19 0)
 			(hide yes)
 			(show_name no)
@@
 	(symbol
 		(lib_id "power:+3.3V")
-		(at 160.02 110.49 0)
+		(at 160.02 115.57 0)
 		(unit 1)
 		(body_style 1)
@@
 		(dnp no)
 		(property "Reference" "#PWR033"
-			(at 160.02 114.3 0)
+			(at 160.02 119.38 0)
 			(hide yes)
 			(show_name no)
@@
 		)
 		(property "Value" "+3.3V"
-			(at 153.67 107.188 0)
+			(at 153.67 112.268 0)
 			(show_name no)
 			(do_not_autoplace no)
@@
 		)
 		(property "Footprint" ""
-			(at 160.02 110.49 0)
+			(at 160.02 115.57 0)
 			(hide yes)
 			(show_name no)
@@
 		)
 		(property "Datasheet" ""
-			(at 160.02 110.49 0)
+			(at 160.02 115.57 0)
 			(hide yes)
 			(show_name no)
@@
 		)
 		(property "Description" "Power symbol creates a global label with name \"+3.3V\""
-			(at 160.02 110.49 0)
-			(hide yes)
-			(show_name no)
+			(at 160.02 115.57 0)
+			(hide yes)
+			(show_name no)
