File: DosingPCB/SolarCharging.kicad_sch (KiCad schematic)
At the start: 30 parts, among them J2 JST, SW2 SW_SPST, U5 BQ25185DLHR, U6 INA260, U7 TPS61022

Commit message: Basically finished schematic
Parts:
- removed U5: BQ25185DLHR, BQ25185DLHR:IC_BQ25185DLHR, symbol BQ25185DLHR:BQ25185DLHR
- added U7: BQ25185DLHR, BQ25185DLHR:IC_BQ25185DLHR, symbol BQ25185DLHR:BQ25185DLHR
- C10: renamed from C8; footprint (none) -> Capacitor_SMD:C_0805_2012Metric
- C11: renamed from C9; footprint (none) -> Capacitor_SMD:C_1206_3216Metric
- C12: renamed from C10; footprint (none) -> Capacitor_SMD:C_1206_3216Metric
- C13: renamed from C11; footprint (none) -> Capacitor_SMD:C_1206_3216Metric
- C14: renamed from C12; footprint (none) -> Capacitor_SMD:C_1206_3216Metric
- C15: renamed from C2; footprint (none) -> Capacitor_SMD:C_0603_1608Metric
- D5: renamed from D6; footprint (none) -> LED_SMD:LED_0603_1608Metric
- D6: renamed from D7; footprint (none) -> LED_SMD:LED_0603_1608Metric
- D7: renamed from D8; footprint (none) -> Diode_SMD:D_SOD-523
- D8: renamed from D10; value Green -> Red; footprint (none) -> LED_SMD:LED_0603_1608Metric
- J7: renamed from J2; footprint Connector_JST:JST_XH_S2B-XH-A_1x02_P2.50mm_Horizontal -> Connector_JST:JST_PH_S2B-PH-K_1x02_P2.00mm_Horizontal
- L1: renamed from L2; footprint (none) -> Inductor_SMD:L_1210_3225Metric
- R12: renamed from R16; footprint (none) -> Resistor_SMD:R_0805_2012Metric
- R13: renamed from R17; footprint (none) -> Resistor_SMD:R_0805_2012Metric
- R14: renamed from R18; footprint (none) -> Resistor_SMD:R_0805_2012Metric
- R15: renamed from R19; footprint (none) -> Resistor_SMD:R_0805_2012Metric
- R16: renamed from R20; footprint (none) -> Resistor_SMD:R_0805_2012Metric
- R17: renamed from R21; footprint (none) -> Resistor_SMD:R_0805_2012Metric
- R18: renamed from R22; footprint (none) -> Resistor_SMD:R_0805_2012Metric
- R19: renamed from R5; footprint (none) -> Resistor_SMD:R_0805_2012Metric
- R20: renamed from R23; footprint (none) -> Resistor_SMD:R_0805_2012Metric
- R21: renamed from R24; footprint (none) -> Resistor_SMD:R_0805_2012Metric
- R22: renamed from R25; footprint (none) -> Resistor_SMD:R_0805_2012Metric
- R23: renamed from R26; footprint (none) -> Resistor_SMD:R_0805_2012Metric
- R24: renamed from R27; footprint (none) -> Resistor_SMD:R_0805_2012Metric
- R25: renamed from R28; footprint (none) -> Resistor_SMD:R_0805_2012Metric
- SW4: renamed from SW2; footprint (none) -> Button_Switch_SMD:SW_SPDT_PCM12
- renumbered U6 to U8, U7 to U9
Connections:
- net +5V: now also U7.4 (~{CE}), U7.5 (GND)
- net V+: now also U7.1 (SYS)
- net at C10.1, D7.1 (K): now also U7.10 (IN)
- net at C12.2, J7.1 (Pin_1), U8.1 (IN+)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: now also U7.2 (BAT)
- net at R13.2: now also U7.9 (STAT1)
- net at R14.1: now also U7.7 (ILIM/VSET)
- net at R15.1, R16.1: now also U7.8 (ISET)
- net at R17.1: now also U7.11 (THERMAL_PAD), U7.6 (TS/MR)
- net at R12.2: now also U7.3 (STAT2)
Other:
- note added: "Check JST size with battery and check pin orientation"
- moved on the sheet: C15

Commit message: 98% completed PCB
Parts:
- removed SW4: SW_SPST, Button_Switch_SMD:SW_SPDT_PCM12, symbol Switch:SW_SPST
- added SW5: SW_SPST, Button_Switch_SMD:SW_SPDT_PCM12, symbol Switch:SW_SPST
Connections:
- net +5V: now also R18.2, SW5.2 (B); no longer C10.2, C11.1, C12.1, C13.1, C14.1, C15.1, C15.2, D8.2 (A), J7.2 (Pin_2), R14.2, R15.2, R16.2, R17.2, R19.1, R19.2, R20.1, R20.2, R23.1, R25.1, U7.4 (~{CE}), U7.5 (GND), U8.10 (VS), U8.11 (GND), U8.14 (IN-), U8.15 (IN-), U8.16 (IN-), U8.4 (A1), U8.5 (A0), U8.6 (GND), U9.1 (GND)
- net Bat_power: now reaches C12.2, J7.1 (Pin_1), U7.2 (BAT), U8.1 (IN+), U8.12 (VBUS), U8.2 (IN+), U8.3 (IN+)
- net at U9.4 (FB): now also R23.2, R25.1; no longer R25.2
- net at U9.3 (VOUT): now also R23.1, SW5.1 (A); no longer R23.2
- new net +3.3V: C15.1, R19.1, R20.1, U8.10 (VS)
- new net GND: C10.2, C11.1, C12.1, C13.1, C14.1, C15.2, D8.2 (A), J7.2 (Pin_2), R14.2, R15.2, R16.2, R17.2, R19.2, R20.2, R25.2, U7.4 (~{CE}), U7.5 (GND), U8.11 (GND), U8.14 (IN-), U8.15 (IN-), U8.16 (IN-), U8.4 (A1), U8.5 (A0), U8.6 (GND), U9.1 (GND)
Other:
- note added: "Adjust resitor (R14, R15, R16) for specific target charging current"
- moved on the sheet: C15, D8, L1, R18, R23, R24, R25, U9

Commit message: Finished PCB - mousebites
Connections:
- net GND: now also U7.11 (THERMAL_PAD)
- net at R17.1, U7.6 (TS/MR): no longer U7.11 (THERMAL_PAD)
Other:
- moved on the sheet: R17
Changed lines of the file:
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@@
 	)
 	(junction
-		(at 189.23 81.28)
+		(at 134.62 92.71)
 		(diameter 0)
 		(color 0 0 0 0)
 	)
 	(junction
-		(at 226.06 113.03)
+		(at 189.23 81.28)
 		(diameter 0)
 		(color 0 0 0 0)
 	)
 	(junction
-		(at 87.63 64.77)
+		(at 226.06 113.03)
 		(diameter 0)
 		(color 0 0 0 0)
 	)
 	(junction
-		(at 134.62 90.17)
+		(at 87.63 64.77)
 		(diameter 0)
 		(color 0 0 0 0)
@@
 	(wire
 		(pts
-			(xy 134.62 80.01) (xy 134.62 90.17)
-		)
-		(stroke
-			(width 0)
-			(type default)
-		)
-	)
-	(wire
-		(pts
 			(xy 149.86 60.96) (xy 149.86 74.93)
 		)
@@
 	(wire
 		(pts
-			(xy 134.62 90.17) (xy 135.89 90.17)
-		)
-		(stroke
-			(width 0)
-			(type default)
-		)
-	)
-	(wire
-		(pts
 			(xy 186.69 44.45) (xy 186.69 48.26)
 		)
@@
 	(wire
 		(pts
+			(xy 134.62 90.17) (xy 134.62 92.71)
+		)
+		(stroke
+			(width 0)
+			(type default)
+		)
+	)
+	(wire
+		(pts
 			(xy 82.55 81.28) (xy 68.58 81.28)
 		)
@@
 	(symbol
 		(lib_id "Device:R")
-		(at 139.7 90.17 90)
+		(at 138.43 80.01 90)
 		(unit 1)
 		(body_style 1)
@@
 		(dnp no)
 		(property "Reference" "R17"
-			(at 141.732 87.63 90)
+			(at 140.462 77.47 90)
 			(show_name no)
 			(do_not_autoplace no)
@@
 		)
 		(property "Value" "10k"
-			(at 141.478 90.17 90)
+			(at 140.208 80.01 90)
 			(show_name no)
 			(do_not_autoplace no)
@@
 		)
 		(property "Footprint" "Resistor_SMD:R_0805_2012Metric"
-			(at 139.7 91.948 90)
+			(at 138.43 81.788 90)
 			(hide yes)
 			(show_name no)
@@
 		)
 		(property "Datasheet" ""
-			(at 139.7 90.17 0)
+			(at 138.43 80.01 0)
 			(hide yes)
 			(show_name no)
@@
 		)
 		(property "Description" "Resistor"
-			(at 139.7 90.17 0)
+			(at 138.43 80.01 0)
 			(hide yes)
 			(show_name no)
@@
 	(symbol
 		(lib_id "power:GND")
-		(at 143.51 90.17 90)
+		(at 142.24 80.01 90)
 		(unit 1)
 		(body_style 1)
@@
 		(fields_autoplaced yes)
 		(property "Reference" "#PWR053"
-			(at 149.86 90.17 0)
+			(at 148.59 80.01 0)
 			(hide yes)
 			(show_name no)
@@
 		)
 		(property "Value" "GND"
-			(at 148.59 90.17 0)
+			(at 147.32 80.01 0)
 			(show_name no)
 			(do_not_autoplace no)
@@
 		)
 		(property "Footprint" ""
-			(at 143.51 90.17 0)
+			(at 142.24 80.01 0)
 			(hide yes)
 			(show_name no)
@@
 		)
 		(property "Datasheet" ""
-			(at 143.51 90.17 0)
+			(at 142.24 80.01 0)
 			(hide yes)
 			(show_name no)
@@
 		)
 		(property "Description" "Power symbol creates a global label with name \"GND\" , ground"
-			(at 143.51 90.17 0)
+			(at 142.24 80.01 0)
 			(hide yes)
 			(show_name no)
