File: DosingPCB/DosingPCB.kicad_pcb (KiCad board)
At the start: 2 copper layers, 71 parts, among them J1 Conn_01x06_Pin, J2 STLink, J3 Servo Conn, J4 SPI header, J5 USB_C_Receptacle_USB2.0_16P, J6 Micro_SD_Card, J7 JST, J8 Solar Cell JST, J9 5V fan JST, Q1 MMBT2222A, SW2 SW_SPDT, SW4 SW_SPST, U1 AMS1117-3.3, U2 STM32L432KBUx, U3 SHTC3, U4 D3V3XA4B10LP, U5 4050, U6 DS3231M, U7 BQ25185DLHR, U8 INA260, U9 TPS61022

Commit message: 98% completed PCB
Parts:
- removed R1: 10k, Resistor_SMD:R_0805_2012Metric
- removed SW4: SW_SPST, Button_Switch_SMD:SW_SPDT_PCM12
- added C16: 10uF, Capacitor_SMD:C_0805_2012Metric, F.Cu at (100.6, 63.1)
- added C17: .1uF, Capacitor_SMD:C_0603_1608Metric, F.Cu at (113.0, 64.8)
- added C25: .1uF, Capacitor_SMD:C_0603_1608Metric, F.Cu at (83.5, 45.3)
- added C26: .1uF, Capacitor_SMD:C_0603_1608Metric, F.Cu at (97.4, 48.8)
- added H4: MountingHole, MountingHole:MountingHole_2.2mm_M2, F.Cu at (150.7, 70.8)
- added H5: MountingHole, MountingHole:MountingHole_2.2mm_M2, F.Cu at (76.5, 48.2)
- added H6: MountingHole, MountingHole:MountingHole_2.2mm_M2, F.Cu at (76.4, 93.3)
- added H7: MountingHole, MountingHole:MountingHole_2.2mm_M2, F.Cu at (176.0, 62.1)
- added H8: MountingHole, MountingHole:MountingHole_2.2mm_M2, F.Cu at (176.1, 79.6)
- added J10: Conn_01x04, Connector_JST:JST_SH_SM04B-SRSS-TB_1x04-1MP_P1.00mm_Horizontal, F.Cu at (170.7, 70.4)
- added J11: Conn_01x04, Connector_JST:JST_SH_SM04B-SRSS-TB_1x04-1MP_P1.00mm_Horizontal, F.Cu at (159.5, 70.7)
- added R26: 10k, Resistor_SMD:R_0805_2012Metric, F.Cu at (112.3, 51.7)
- added SW1: SW_Push, Button_Switch_SMD:SW_Push_SPST_NO_Alps_SKRK, F.Cu at (45.9, 76.8)
- added SW3: SW_Push, Button_Switch_SMD:SW_Push_SPST_NO_Alps_SKRK, F.Cu at (69.1, 46.5)
- added SW5: SW_SPST, Button_Switch_SMD:SW_SPDT_PCM12, F.Cu at (107.2, 95.9)
- J1: footprint Connector_PinHeader_1.00mm:PinHeader_1x06_P1.00mm_Vertical -> Connector_PinHeader_2.54mm:PinHeader_1x06_P2.54mm_Vertical
- J2: footprint Connector_PinHeader_1.00mm:PinHeader_1x02_P1.00mm_Vertical -> Connector_PinHeader_2.54mm:PinHeader_1x02_P2.54mm_Vertical
- J3: footprint Connector_PinHeader_1.00mm:PinHeader_1x03_P1.00mm_Horizontal -> Connector_PinHeader_2.54mm:PinHeader_1x03_P2.54mm_Horizontal
- J4: footprint Connector_PinHeader_1.00mm:PinHeader_1x08_P1.00mm_Vertical -> Connector_PinHeader_2.54mm:PinHeader_1x08_P2.54mm_Vertical
- moved J8 126.7 mm to (48.9, 94.0), turned to -90 degrees
- moved J7 124.2 mm to (48.9, 84.7), turned to -90 degrees
- moved D7 122.5 mm to (53.6, 94.0), turned to 180 degrees
- moved C12 113.6 mm to (54.1, 83.1), turned to 90 degrees
- moved D6 104.6 mm to (59.2, 90.0), turned to 90 degrees
- moved U7 103.2 mm to (71.7, 89.4), turned to 180 degrees
- moved C2 101.5 mm to (51.6, 77.0), turned to -90 degrees
- moved C11 97.4 mm to (69.9, 96.2), turned to 90 degrees
- moved C10 95.2 mm to (59.4, 96.0), turned to 180 degrees
- moved R15 91.0 mm to (64.2, 81.1), turned to 90 degrees
- moved R16 90.0 mm to (64.9, 85.5), turned to 180 degrees
- moved D5 89.3 mm to (76.0, 81.9), turned to 90 degrees
- moved R13 89.3 mm to (64.1, 89.8), turned to 90 degrees
- moved D1 87.0 mm to (84.5, 56.7), turned to 180 degrees
- moved R17 86.4 mm to (71.5, 85.8)
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Connections:
- net /Solar+Charging/VIN/Solar+ renamed /Solar_power
- net Net-(J7-Pin_1) renamed /Solar+Charging/Bat_power
- BT1 pad 2: +5V -> GND
- C1 pad 2: +5V -> GND
- C10 pad 2: +5V -> GND
- C11 pad 1: +5V -> GND
- C12 pad 1: +5V -> GND
- C13 pad 1: +5V -> GND
- C14 pad 1: +5V -> GND
- C15 pad 1: +5V -> +3.3V
- C15 pad 2: +5V -> GND
- C2 pad 1: +5V -> GND
- C3 pad 2: +5V -> GND
- C4 pad 2: +5V -> GND
- C5 pad 2: +5V -> GND
- C6 pad 2: +5V -> GND
- C7 pad 2: +5V -> GND
- C8 pad 2: +5V -> GND
- C9 pad 1: +5V -> GND
- D8 pad 2: +5V -> GND
- J1 pad 1: +5V -> GND
- J1 pad 4: Net-(J1-Pin_4) -> header conn
- J3 pad 2: +3.3V -> +5V
- J3 pad 3: +5V -> GND
- J4 pad 1: +5V -> GND
- J5 pad A1: +5V -> GND
- J5 pad A12: +5V -> GND
- J5 pad B1: +5V -> GND
- J5 pad B12: +5V -> GND
- J5 pad SH: +5V -> GND
- J6 pad 6: +5V -> GND
- J6 pad SH: +5V -> GND
- J7 pad 2: +5V -> GND
- J8 pad 2: +5V -> GND
- Q1 pad 2: +5V -> GND
- R14 pad 2: +5V -> GND
- R15 pad 2: +5V -> GND
- R16 pad 2: +5V -> GND
- R17 pad 2: +5V -> GND
- R18 pad 2: Net-(SW4-A) -> +5V
- R19 pad 1: +5V -> +3.3V
- R19 pad 2: +5V -> GND
- R2 pad 2: +5V -> GND
- R20 pad 1: +5V -> +3.3V
- R20 pad 2: +5V -> GND
- R21 pad 2: RTC_SCL -> RTC_SDA
- R23 pad 1: +5V -> Net-(SW5-A)
- R23 pad 2: Net-(U9-VOUT) -> Net-(U9-FB)
- R25 pad 1: +5V -> Net-(U9-FB)
- R25 pad 2: Net-(U9-FB) -> GND
- R4 pad 1: Temp_SDA -> Temp_SCL
- R5 pad 1: Temp_SCL -> Temp_SDA
- R6 pad 2: +5V -> GND
- R7 pad 2: +5V -> GND
- SW2 pad 1: +5V -> GND
- U1 pad 1: +5V -> GND
- U2 pad 14: Net-(J1-Pin_4) -> CD
- U2 pad 16: +5V -> GND
- U2 pad 31: Net-(U2-PH3) -> Net-(SW2-B)
- U2 pad 32: +5V -> GND
- U2 pad 33: +5V -> GND
- U2 pad 6: CD -> header conn
- U3 pad 2: Temp_SCL -> Temp_SDA
- U3 pad 3: Temp_SDA -> Temp_SCL
- U3 pad 4: +5V -> GND
- U4 pad 3: +5V -> GND
- U4 pad 8: +5V -> GND
- U5 pad 11: +5V -> GND
- U5 pad 14: +5V -> GND
- U5 pad 8: +5V -> GND
- U6 pad 13: +5V -> GND
- U7 pad 4: +5V -> GND
- U7 pad 5: +5V -> GND
- U8 pad 10: +5V -> +3.3V
- U8 pad 11: +5V -> GND
- U8 pad 14: +5V -> GND
- U8 pad 15: +5V -> GND
- U8 pad 16: +5V -> GND
- U8 pad 4: +5V -> GND
- U8 pad 5: +5V -> GND
- U8 pad 6: +5V -> GND
- U9 pad 1: +5V -> GND
- U9 pad 3: Net-(U9-VOUT) -> Net-(SW5-A)
Routing:
- net GND: track 0.00 -> 189.3 mm, vias 0 -> 49
- net RTC_SDA: track 0.00 -> 147.7 mm, vias 0 -> 4
- net RTC_SCL: track 0.00 -> 142.9 mm, vias 0 -> 4
- net CD: track 0.00 -> 112.6 mm, vias 0 -> 2
- net +3.3V: track 0.00 -> 87.3 mm, vias 0 -> 23
- net /Solar+Charging/Bat_power: track 0.00 -> 81.4 mm
- net SD_CLK: track 0.00 -> 64.5 mm
- net V+: track 0.00 -> 62.4 mm, vias 0 -> 4
- net Net-(U2-NRST): track 0.00 -> 60.5 mm
- net SD_DataIn: track 0.00 -> 54.1 mm, vias 0 -> 2
- net CS: track 0.00 -> 53.2 mm
- net Data+: track 0.00 -> 52.5 mm, vias 0 -> 2
- net Data-: track 0.00 -> 52.1 mm
- net Net-(J9-Pin_1): track 0.00 -> 46.4 mm
- net Net-(J1-Pin_3): track 0.00 -> 44.7 mm, vias 0 -> 1
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- added copper zone on In2.Cu, net +3.3V
- added copper zone on In2.Cu, net +5V
- added copper zone on In1.Cu, net GND
- added copper zone on In2.Cu, net V+
Other:
- board outline added: 142.5 x 57.1 mm
- copper layers 2 -> 4
- board text added: "- Look at picture for connectors - check sizes for JSTs"
- board text added: "- Snap off temp - 40mm x 160 ish mm"

Commit message: Finished PCB - mousebites
Parts:
- added REF**: BreakLine_11h_D0.5mm_P0.85mm, Panelization:BreakLine_11h_D0.5mm_P0.85mm, F.Cu at (163.4, 66.8)
- added REF**: BreakLine_11h_D0.5mm_P0.85mm, Panelization:BreakLine_11h_D0.5mm_P0.85mm, F.Cu at (166.8, 76.1)
- added REF**: BreakLine_11h_D0.5mm_P0.85mm, Panelization:BreakLine_11h_D0.5mm_P0.85mm, F.Cu at (163.4, 76.1)
- added REF**: BreakLine_11h_D0.5mm_P0.85mm, Panelization:BreakLine_11h_D0.5mm_P0.85mm, F.Cu at (166.8, 66.8)
- moved C3 9.19 mm to (87.3, 68.5)
- moved BT1 0.85 mm to (52.8, 58.1)
- moved R4 0.55 mm to (180.3, 72.8)
- moved R5 0.55 mm to (180.3, 67.6)
Connections:
- J1 pad 4: header conn -> unconnected-(J1-Pin_4-Pad4)
- J1 pad 5: Net-(J1-Pin_5) -> unconnected-(J1-Pin_5-Pad5)
- U2 pad 15: Net-(J1-Pin_5) -> unconnected-(U2-PB1-Pad15)
- U2 pad 6: header conn -> unconnected-(U2-PA0-Pad6)
Routing:
- net SD_DataOut: track 0.00 -> 63.7 mm, vias 0 -> 4
- net Temp_SCL: track 8.15 -> 70.9 mm, vias 0 -> 2
- net Temp_SDA: track 7.91 -> 69.9 mm, vias 0 -> 2
- net Net-(BT1-+): track 31.6 -> 53.8 mm
- net Net-(D4-A): track 0.00 -> 13.5 mm, vias 0 -> 2
- net +3.3V: track 87.3 -> 100.5 mm, vias 23 -> 27
- net GND: track 189.3 -> 198.9 mm, vias 49 -> 51
- net +5V: track 24.2 -> 19.9 mm, vias 9 -> 8
- net Net-(U2-PA2): track 33.2 -> 30.4 mm
- net Net-(J6-CMD): track 31.0 -> 29.1 mm
- net Net-(U6-~{RST}): track 17.9 -> 17.1 mm
- net Net-(J5-D--PadA7): track 15.5 -> 16.3 mm

Commit message: error fixes + logo
Parts:
- added REF**: MiteOut_Logo, Logo:MiteOut_Logo, F.Cu at (130.4, 44.4)
- moved J11 0.29 mm to (159.8, 70.7)
- moved J10 0.25 mm to (170.4, 70.4)
Connections:
- R17 pad 1: Net-(U7-THERMAL_PAD) -> Net-(U7-TS/MR)
- U7 pad 11: Net-(U7-THERMAL_PAD) -> GND
- U7 pad 12: (no net) -> GND
- U7 pad 13: (no net) -> GND
- U7 pad 6: Net-(U7-THERMAL_PAD) -> Net-(U7-TS/MR)
Routing:
- net Net-(U7-THERMAL_PAD): track 4.31 -> 0.00 mm
- net Net-(U7-TS/MR): track 0.00 -> 2.85 mm
- net Temp_SDA: track 69.9 -> 70.8 mm
- net RTC_SCL: track 143.3 -> 142.7 mm
- added copper zone on B.Cu, net V+
- removed copper zone on In2.Cu, net V+
Other:
- outline, holes or cut-outs redrawn
- board text added: "MITE OUT"
- board text removed: "- Look at picture for connectors - check sizes for JSTs"
- board text removed: "- Snap off temp - 40mm x 160 ish mm"
